Commit message: Create biped task

File: assets/urdf/biped/urdf/biped.urdf (robot description, URDF)
Before this commit: robot biped, 9 links, 8 joints
Links:
- link abad_L_Link: geometry visual mesh filename=../meshes/abad_left_link.STL
- link abad_R_Link: geometry visual mesh filename=../meshes/abad_right_link.STL
- link hip_L_Link: geometry visual mesh filename=../meshes/hip_left_link.STL
- link hip_R_Link: geometry visual mesh filename=../meshes/hip_right_link.STL
